File: Connectors.kicad_sch (KiCad schematic)
At the start: 4 parts, among them J1 Conn_01x04_Pin, J2 Conn_01x04_Pin, J3 Conn_01x09_Pin, J4 Conn_02x03_Odd_Even

Commit message: assign footprints
Parts:
- J1, J2: footprint (none) -> Connector_PinHeader_2.54mm:PinHeader_1x04_P2.54mm_Vertical
- J3: footprint (none) -> Connector_PinHeader_2.54mm:PinHeader_1x09_P2.54mm_Vertical
- J4: footprint (none) -> Connector_PinHeader_2.54mm:PinHeader_2x03_P2.54mm_Vertical
Changed lines of the file:
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@@
 			)
 		)
-		(property "Footprint" ""
+		(property "Footprint" "Connector_PinHeader_2.54mm:PinHeader_1x04_P2.54mm_Vertical"
 			(at 143.51 105.41 0)
 			(hide yes)
@@
 			)
 		)
-		(property "Footprint" ""
+		(property "Footprint" "Connector_PinHeader_2.54mm:PinHeader_1x09_P2.54mm_Vertical"
 			(at 144.145 132.715 0)
 			(hide yes)
@@
 			)
 		)
-		(property "Footprint" ""
+		(property "Footprint" "Connector_PinHeader_2.54mm:PinHeader_2x03_P2.54mm_Vertical"
 			(at 170.815 130.81 0)
 			(hide yes)
@@
 			)
 		)
-		(property "Footprint" ""
+		(property "Footprint" "Connector_PinHeader_2.54mm:PinHeader_1x04_P2.54mm_Vertical"
 			(at 166.37 104.775 0)
 			(hide yes)

Commit message: finish schematic
Parts:
- renumbered J3 to J2, J2 to J3
Connections:
- net GND: now reaches J1.1 (Pin_1)
- net GND: now also J2.8 (Pin_8), J3.1 (Pin_1), J4.6 (Pin_6)
- net Vcc: now reaches J1.2 (Pin_2)
- net Vcc: now also J2.9 (Pin_9), J3.2 (Pin_2), J4.2 (Pin_2)
- net SDA: now reaches J1.3 (Pin_3)
- net SCL: now reaches J1.4 (Pin_4)
- net D2: now reaches J2.1 (Pin_1)
- net D3: now reaches J2.2 (Pin_2)
- net D4: now reaches J2.3 (Pin_3)
- net D5: now reaches J2.4 (Pin_4)
- net D6: now reaches J2.5 (Pin_5)
- net D7: now reaches J2.6 (Pin_6)
- net D8: now reaches J2.7 (Pin_7)
- net MISO: now reaches J4.1 (Pin_1)
- net SCK: now reaches J4.3 (Pin_3)
- net MOSI: now reaches J4.4 (Pin_4)
- net RST: now reaches J4.5 (Pin_5)
- net RX: now reaches J3.3 (Pin_3)
- net TX: now reaches J3.4 (Pin_4)
Changed lines of the file:
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@@
 	(generator_version "10.0")
 	(paper "A4")
+	(hierarchical_label "Vcc"
+		(shape passive)
+		(at 149.225 142.875 0)
+		(effects
+			(font
+				(size 1.27 1.27)
+			)
+			(justify left)
+		)
+	)
+	(hierarchical_label "MOSI"
+		(shape input)
+		(at 178.435 130.81 0)
+		(effects
+			(font
+				(size 1.27 1.27)
+			)
+			(justify left)
+		)
+	)
+	(hierarchical_label "MISO"
+		(shape output)
+		(at 165.735 128.27 180)
+		(effects
+			(font
+				(size 1.27 1.27)
+			)
+			(justify right)
+		)
+	)
+	(hierarchical_label "SCK"
+		(shape passive)
+		(at 165.735 130.81 180)
+		(effects
+			(font
+				(size 1.27 1.27)
+			)
+			(justify right)
+		)
+	)
+	(hierarchical_label "Vcc"
+		(shape passive)
+		(at 171.45 104.775 0)
+		(effects
+			(font
+				(size 1.27 1.27)
+			)
+			(justify left)
+		)
+	)
+	(hierarchical_label "RX"
+		(shape input)
+		(at 171.45 107.315 0)
+		(effects
+			(font
+				(size 1.27 1.27)
+			)
+			(justify left)
+		)
+	)
+	(hierarchical_label "D7"
+		(shape bidirectional)
+		(at 149.225 135.255 0)
+		(effects
+			(font
+				(size 1.27 1.27)
+			)
+			(justify left)
+		)
+	)
+	(hierarchical_label "Vcc"
+		(shape passive)
+		(at 148.59 105.41 0)
+		(effects
+			(font
+				(size 1.27 1.27)
+			)
+			(justify left)
+		)
+	)
+	(hierarchical_label "D2"
+		(shape bidirectional)
+		(at 149.225 122.555 0)
+		(effects
+			(font
+				(size 1.27 1.27)
+			)
+			(justify left)
+		)
+	)
+	(hierarchical_label "RST"
+		(shape passive)
+		(at 165.735 133.35 180)
+		(effects
+			(font
+				(size 1.27 1.27)
+			)
+			(justify right)
+		)
+	)
+	(hierarchical_label "D4"
+		(shape bidirectional)
+		(at 149.225 127.635 0)
+		(effects
+			(font
+				(size 1.27 1.27)
+			)
+			(justify left)
+		)
+	)
+	(hierarchical_label "D6"
+		(shape bidirectional)
+		(at 149.225 132.715 0)
+		(effects
+			(font
+				(size 1.27 1.27)
+			)
+			(justify left)
+		)
+	)
+	(hierarchical_label "GND"
+		(shape passive)
+		(at 178.435 133.35 0)
+		(effects
+			(font
+				(size 1.27 1.27)
+			)
+			(justify left)
+		)
+	)
+	(hierarchical_label "D3"
+		(shape bidirectional)
+		(at 149.225 125.095 0)
+		(effects
+			(font
+				(size 1.27 1.27)
+			)
+			(justify left)
+		)
+	)
+	(hierarchical_label "D5"
+		(shape bidirectional)
+		(at 149.225 130.175 0)
+		(effects
+			(font
+				(size 1.27 1.27)
+			)
+			(justify left)
+		)
+	)
+	(hierarchical_label "D8"
+		(shape bidirectional)
+		(at 149.225 137.795 0)
+		(effects
+			(font
+				(size 1.27 1.27)
+			)
+			(justify left)
+		)
+	)
+	(hierarchical_label "SDA"
+		(shape bidirectional)
+		(at 148.59 107.95 0)
+		(effects
+			(font
+				(size 1.27 1.27)
+			)
+			(justify left)
+		)
+	)
+	(hierarchical_label "Vcc"
+		(shape passive)
+		(at 178.435 128.27 0)
+		(effects
+			(font
+				(size 1.27 1.27)
+			)
+			(justify left)
+		)
+	)
+	(hierarchical_label "SCL"
+		(shape passive)
+		(at 148.59 110.49 0)
+		(effects
+			(font
+				(size 1.27 1.27)
+			)
+			(justify left)
+		)
+	)
+	(hierarchical_label "TX"
+		(shape output)
+		(at 171.45 109.855 0)
+		(effects
+			(font
+				(size 1.27 1.27)
+			)
+			(justify left)
+		)
+	)
+	(hierarchical_label "GND"
+		(shape passive)
+		(at 171.45 102.235 0)
+		(effects
+			(font
+				(size 1.27 1.27)
+			)
+			(justify left)
+		)
+	)
+	(hierarchical_label "GND"
+		(shape passive)
+		(at 149.225 140.335 0)
+		(effects
+			(font
+				(size 1.27 1.27)
+			)
+			(justify left)
+		)
+	)
+	(hierarchical_label "GND"
+		(shape passive)
+		(at 148.59 102.87 0)
+		(effects
+			(font
+				(size 1.27 1.27)
+			)
+			(justify left)
+		)
+	)
 	(symbol
 		(lib_id "Connector:Conn_01x04_Pin")
@@
 		(in_pos_files yes)
 		(dnp no)
-		(property "Reference" "J3"
+		(property "Reference" "J2"
 			(at 144.78 117.475 0)
 			(show_name no)
@@
 			(project "MCU Datalogger"
 				(path "/6ab5cb73-b588-47d2-abf7-17ca87af1645/dc577c61-1aa5-4e02-9855-2ed2eccfa9a4"
-					(reference "J3")
+					(reference "J2")
 					(unit 1)
 				)
@@
 		(in_pos_files yes)
 		(dnp no)
-		(property "Reference" "J2"
+		(property "Reference" "J3"
 			(at 167.005 97.79 0)
 			(show_name no)
@@
 			(project "MCU Datalogger"
 				(path "/6ab5cb73-b588-47d2-abf7-17ca87af1645/dc577c61-1aa5-4e02-9855-2ed2eccfa9a4"
-					(reference "J2")
+					(reference "J3")
 					(unit 1)
 				)
